File: cmos_nand_dflip/cmos_nand_dflip.sch (KiCad schematic (older format))
At the start: 11 parts, among them X1 CMOS_NAND, X2 CMOS_NAND, X3 CMOS_NAND, X4 CMOS_NAND, X5 CMOS_NAND, X6 CMOS_NAND

Commit message: Change file path for spice_models.lib to relative path (seems to work)
Parts:
- X1, X2, X3, X4, X5, X6: Spice_Lib_File C:\\temp3\\spice_v5\\libs\\spice_models.lib -> ../libs/spice_models.lib
Changed lines of the file:
@@
 F 5 "NAND" H 6200 3500 50  0001 C CNN "Spice_Model"
 F 6 "Y" H 6200 3500 50  0001 C CNN "Spice_Netlist_Enabled"
-F 7 "C:\\temp3\\spice_v5\\libs\\spice_models.lib" H 6200 3500 50  0001 C CNN "Spice_Lib_File"
+F 7 "../libs/spice_models.lib" H 6200 3500 50  0001 C CNN "Spice_Lib_File"
 	1    6200 3500
 	1    0    0    -1
@@
 F 5 "NAND" H 4900 3400 50  0001 C CNN "Spice_Model"
 F 6 "Y" H 4900 3400 50  0001 C CNN "Spice_Netlist_Enabled"
-F 7 "C:\\temp3\\spice_v5\\libs\\spice_models.lib" H 4900 3400 50  0001 C CNN "Spice_Lib_File"
+F 7 "../libs/spice_models.lib" H 4900 3400 50  0001 C CNN "Spice_Lib_File"
 	1    4900 3400
 	1    0    0    -1
@@
 F 5 "NAND3" H 4900 4800 50  0001 C CNN "Spice_Model"
 F 6 "Y" H 4900 4800 50  0001 C CNN "Spice_Netlist_Enabled"
-F 7 "C:\\temp3\\spice_v5\\libs\\spice_models.lib" H 4900 4800 50  0001 C CNN "Spice_Lib_File"
+F 7 "../libs/spice_models.lib" H 4900 4800 50  0001 C CNN "Spice_Lib_File"
 	1    4900 4800
 	1    0    0    -1
@@
 F 5 "NAND" H 6200 4700 50  0001 C CNN "Spice_Model"
 F 6 "Y" H 6200 4700 50  0001 C CNN "Spice_Netlist_Enabled"
-F 7 "C:\\temp3\\spice_v5\\libs\\spice_models.lib" H 6200 4700 50  0001 C CNN "Spice_Lib_File"
+F 7 "../libs/spice_models.lib" H 6200 4700 50  0001 C CNN "Spice_Lib_File"
 	1    6200 4700
 	1    0    0    -1
@@
 F 5 "NAND" H 4900 2200 50  0001 C CNN "Spice_Model"
 F 6 "Y" H 4900 2200 50  0001 C CNN "Spice_Netlist_Enabled"
-F 7 "C:\\temp3\\spice_v5\\libs\\spice_models.lib" H 4900 2200 50  0001 C CNN "Spice_Lib_File"
+F 7 "../libs/spice_models.lib" H 4900 2200 50  0001 C CNN "Spice_Lib_File"
 	1    4900 2200
 	1    0    0    -1
@@
 F 5 "NAND" H 4900 6000 50  0001 C CNN "Spice_Model"
 F 6 "Y" H 4900 6000 50  0001 C CNN "Spice_Netlist_Enabled"
-F 7 "C:\\temp3\\spice_v5\\libs\\spice_models.lib" H 4900 6000 50  0001 C CNN "Spice_Lib_File"
+F 7 "../libs/spice_models.lib" H 4900 6000 50  0001 C CNN "Spice_Lib_File"
 	1    4900 6000
 	1    0    0    -1
