File: cmos_nand_sub/cmos_nand_sub.sch (KiCad schematic (older format))
At the start: 5 parts, among them X1 CMOS_NAND

Commit message: Change file path for spice_models.lib to relative path (seems to work)
Parts:
- X1: Spice_Lib_File C:\\temp3\\spice_v5\\libs\\spice_models.lib -> ../libs/spice_models.lib
Changed lines of the file:
@@
 F 5 "NAND" H 5500 3350 50  0001 C CNN "Spice_Model"
 F 6 "Y" H 5500 3350 50  0001 C CNN "Spice_Netlist_Enabled"
-F 7 "C:\\temp3\\spice_v5\\libs\\spice_models.lib" H 5500 3350 50  0001 C CNN "Spice_Lib_File"
+F 7 "../libs/spice_models.lib" H 5500 3350 50  0001 C CNN "Spice_Lib_File"
 	1    5500 3350
 	1    0    0    -1
